Commit message: Working gripper controller Add fake joint for ee

File: ur_robotiq_isaac/urdfs/ur5e_robotiq.urdf (robot description, URDF)
Before this commit: robot ur5e, 24 links, 23 joints
Links:
- added link gripper_ee
Joints:
- added joint gripper_ee_joint: type fixed, parent robotiq_arg2f_base_link, child gripper_ee, origin xyz=0 0 0.2 rpy=0 0 0

File: ur_robotiq_isaac/urdfs/ur5e_robotiq.xacro (robot description, xacro)
@@ -112,4 +112,10 @@
       <child link="$(arg robotiq_prefix)robotiq_arg2f_base_link" />
     </joint>
+    <link name="gripper_ee"/>
+    <joint name="gripper_ee_joint" type="fixed">
+      <origin xyz="0 0 0.2" rpy="0 0 0" />
+      <parent link="$(arg robotiq_prefix)robotiq_arg2f_base_link" />
+      <child link="gripper_ee" />
+    </joint>
     <xacro:include filename="$(find robotiq_2f_140_gripper_visualization)/urdf/robotiq_arg2f_140_model_macro.xacro" />
     <xacro:robotiq_arg2f_140 prefix=""/>
@@ -121,4 +127,10 @@
       <child link="$(arg robotiq_prefix)robotiq_arg2f_base_link" />
     </joint>
+    <link name="gripper_ee"></link>
+    <joint name="gripper_ee_joint" type="fixed">
+      <origin xyz="0 0 0.2" rpy="0 0 0" />
+      <parent link="$(arg robotiq_prefix)robotiq_arg2f_base_link" />
+      <child link="$(arg robotiq_prefix)tool_to_gripper" />
+    </joint>
     <xacro:include filename="$(find robotiq_2f_85_gripper_visualization)/urdf/robotiq_arg2f_85_model_macro.xacro" />
     <xacro:robotiq_arg2f_85 prefix=""/>

Commit message: Update collision

File: ur_robotiq_isaac/urdfs/ur5e_robotiq.urdf (robot description, URDF)
Before this commit: robot ur5e, 25 links, 24 joints
Joints:
- joint gripper_ee_joint: origin xyz=0 0 0.2 rpy=0 0 0 -> xyz=0 0 0.235 rpy=0 0 0

File: ur_robotiq_isaac/urdfs/ur5e_robotiq.xacro (robot description, xacro)
@@ -114,5 +114,5 @@
     <link name="gripper_ee"/>
     <joint name="gripper_ee_joint" type="fixed">
-      <origin xyz="0 0 0.2" rpy="0 0 0" />
+      <origin xyz="0 0 0.235" rpy="0 0 0" />
       <parent link="$(arg robotiq_prefix)robotiq_arg2f_base_link" />
       <child link="gripper_ee" />
@@ -129,5 +129,5 @@
     <link name="gripper_ee"></link>
     <joint name="gripper_ee_joint" type="fixed">
-      <origin xyz="0 0 0.2" rpy="0 0 0" />
+      <origin xyz="0 0 0.235" rpy="0 0 0" />
       <parent link="$(arg robotiq_prefix)robotiq_arg2f_base_link" />
       <child link="$(arg robotiq_prefix)tool_to_gripper" />

Commit message: Add Joints limit to UR

File: ur_robotiq_isaac/urdfs/ur5e_robotiq.urdf (robot description, URDF)
Before this commit: robot ur5e, 25 links, 24 joints
Joints:
- joint elbow_joint: limit lower=-3.141592653589793 upper=3.141592653589793 effort=150.0 velocity=3.141592653589793 -> lower=-2.618 upper=0.2618 effort=150.0 velocity=3.141592653589793
- joint shoulder_pan_joint: limit lower=-6.283185307179586 upper=6.283185307179586 effort=150.0 velocity=3.141592653589793 -> lower=-6.283185307179586 upper=3.49 effort=150.0 velocity=3.141592653589793
- joint wrist_1_joint: limit lower=-6.283185307179586 upper=6.283185307179586 effort=28.0 velocity=3.141592653589793 -> lower=-5.58505 upper=3.31613 effort=28.0 velocity=3.141592653589793
- joint wrist_2_joint: limit lower=-6.283185307179586 upper=6.283185307179586 effort=28.0 velocity=3.141592653589793 -> lower=-1.74533 upper=3.14159 effort=28.0 velocity=3.141592653589793

Commit message: Safer Limits

File: ur_robotiq_isaac/urdfs/ur5e_robotiq.urdf (robot description, URDF)
Before this commit: robot ur5e, 25 links, 24 joints
Joints:
- joint elbow_joint: limit lower=-2.618 upper=0.2618 effort=150.0 velocity=3.141592653589793 -> lower=-2.44 upper=0.2618 effort=150.0 velocity=3.141592653589793
